Commit message: Fix gazebo loading and rviz tf problem

File: robot_description/urdf/Assem2.SLDASM.urdf (robot description, URDF)
Before this commit: robot Assem2.SLDASM, 5 links, 4 joints
Links:
- added link lidar2d_link, mass 0.2; collision box size=0.02 0.02 0.02; visual box size=0.02 0.02 0.02
Joints:
- added joint lidar2d_joint: type fixed, parent base_link, child lidar2d_link, origin xyz=0.0 0.0 0.1 rpy=0.0 0.0 0.0
